File: hardware/gbflasher.sch (KiCad schematic (older format))
At the start: 33 parts, among them IC1 ATTINY2313-P, J1 USB, P1 CONN_5X2, P2 GB_CART_CONN, P3 CONN_5, P4 CONN_2, U1 74LS574, U2 74LS574, U3 FT230XS

Commit message: Added license
Parts:
- U1, U2: value 74LS574 -> 74HCT573; symbol 74LS574 -> 74LS573
Changed lines of the file:
@@
 LIBS:contrib
 LIBS:valves
-LIBS:ft230xs
 LIBS:gbflasher-cache
 EELAYER 27 0
@@
 $EndComp
 $Comp
-L 74LS574 U2
+L 74LS573 U2
 U 1 1 5528163B
 P 2850 7950
 F 0 "U2" H 2850 7950 60  0000 C CNN
-F 1 "74LS574" H 2900 7600 60  0000 C CNN
+F 1 "74HCT573" H 2900 7600 60  0000 C CNN
 F 2 "" H 2850 7950 60  0001 C CNN
 F 3 "" H 2850 7950 60  0001 C CNN
@@
 $EndComp
 $Comp
-L 74LS574 U1
+L 74LS573 U1
 U 1 1 55281634
 P 2850 6200
 F 0 "U1" H 2850 6200 60  0000 C CNN
-F 1 "74LS574" H 2900 5850 60  0000 C CNN
+F 1 "74HCT573" H 2900 5850 60  0000 C CNN
 F 2 "" H 2850 6200 60  0001 C CNN
 F 3 "" H 2850 6200 60  0001 C CNN
